File: Car_Circuit/Car_Circuit.kicad_sch (KiCad schematic)
At the start: 2 parts

Commit message: Update car wiring diagram
Parts:
- added Brake, Diff_swich, KSW1: SW_DPST_x2, symbol Switch:SW_DPST_x2
- added Deutsch_connector: ~, symbol Car_Parts _library:Deutsch_8_way_connect
- added Diff: ~, symbol Car_Parts _library:Diff
- added Engine: ~, symbol Car_Parts _library:Engine
- added U2, U3: ~, symbol Car_Parts _library:Power_Bus
Connections:
- net GND: now also KSW1.2 (B), KSW1.4 (B), U3. (Vout_4); no longer U1.3 (GND)
- net at BT1.1 (+): now also U2. (Vout_4)
- net at U1.2 (Stop): now also Deutsch_connector.6 (Output_6)
- new net: Engine. (Spark), KSW1.1 (A), KSW1.3 (A)
- new net: U1.3 (GND), U3. (Vout_4)
- new net: Deutsch_connector.8 (Output_8), U3. (Vout_4)
- new net: Deutsch_connector.1 (Output_1), U2. (Vout_4)
- new net: Deutsch_connector.2 (Output_2), U2. (Vout_4)
- new net: Brake.3 (A), Deutsch_connector.6 (Output_6)
- new net: Brake.4 (B), Deutsch_connector.2 (Output_2)
- new net: Deutsch_connector.1 (Output_1), Diff_swich.2 (B)
- new net: Deutsch_connector.8 (Output_8), Diff.2 (Gnd)
- new net: Diff.1 (Vin), Diff_swich.1 (A)
Other:
- moved on the sheet: BT1, U1
